Commit message: Moveit2 fetch setup

File: urdf/fetch_2.urdf (robot description, URDF)
Before this commit: robot fetch, 26 links, 25 joints
Links:
- removed link bellows_link
- removed link head_camera_depth_frame
- removed link head_camera_depth_optical_frame
- removed link head_camera_link
- removed link head_camera_rgb_frame
- removed link head_camera_rgb_optical_frame
- link base_link: geometry collision cylinder length=0.33 radius=0.28; visual mesh filename=package://fetch/meshes/base_link.dae
- link estop_link: geometry collision mesh filename=package://fetch/meshes/estop_link.STL; visual mesh filename=package://fetch/meshes/estop_link.STL
- link l_gripper_finger_link: geometry collision box size=0.062 0.013 0.026; visual mesh filename=package://fetch/meshes/l_gripper_finger_link.STL
- link l_wheel_link: geometry collision sphere radius=0.065; visual mesh filename=package://fetch/meshes/l_wheel_link.STL
- link r_gripper_finger_link: geometry collision box size=0.062 0.013 0.026; visual mesh filename=package://fetch/meshes/r_gripper_finger_link.STL
- link r_wheel_link: geometry collision sphere radius=0.065; visual mesh filename=package://fetch/meshes/r_wheel_link.STL
Joints:
- removed joint bellows_joint
- removed joint head_camera_depth_joint
- removed joint head_camera_depth_optical_joint
- removed joint head_camera_joint
- removed joint head_camera_rgb_joint
- removed joint head_camera_rgb_optical_joint
