Commit message: Fixed ros2_control xacro

File: fetch_description/urdf/fetch.urdf (robot description, URDF)
Before this commit: robot fetch, 27 links, 26 joints
Links:
- removed link fetch_tool_link
Joints:
- removed joint fetch_tool_fixed_joint

File: fetch_moveit_config/config/fetch.ros2_control.xacro (robot description, xacro)
@@ -4,8 +4,16 @@
         <xacro:property name="initial_positions" value="${load_yaml(initial_positions_file)['initial_positions']}"/>
         <ros2_control name="${name}" type="system">
-            <hardware>
-                <!-- By default, set up controllers for simulation. This won't work on real hardware -->
-                <plugin>mock_components/GenericSystem</plugin>
+	     <hardware>
+                    <plugin>topic_based_ros2_control/TopicBasedSystem</plugin>
+                    <param name="joint_commands_topic">/isaac_joint_commands</param>
+                    <param name="joint_states_topic">/isaac_joint_states</param>
             </hardware>
+            <joint name="shoulder_pan_joint">
+                <command_interface name="position"/>
+                <state_interface name="position">
+                  <param name="initial_value">${initial_positions['shoulder_pan_joint']}</param>
+                </state_interface>
+                <state_interface name="velocity"/>
+            </joint>
             <joint name="shoulder_lift_joint">
                 <command_interface name="position"/>

Commit message: Bucket congfig, need to fix launch

File: fetch_description/urdf/fetch.urdf (robot description, URDF)
Before this commit: robot fetch, 26 links, 25 joints
Links:
- added link fetch_tool_link; collision mesh filename=package://fetch_description/meshes/bucket.STL scale=0.001 0.001 0.001; visual mesh filename=package://fetch_description/meshes/bucket.STL scale=0.01 0.01 0.01
Joints:
- added joint fetch_tool_fixed_joint: type fixed, parent gripper_link, child fetch_tool_link, origin xyz=-0.1 0 -0.195 rpy=0 1.5708 0

Commit message: SVD I

File: fetch_description/urdf/fetch.urdf (robot description, URDF)
Before this commit: robot fetch, 26 links, 25 joints
Links:
- added link fetch_tool_link; collision mesh filename=package://fetch_description/meshes/bucket.STL scale=0.01 0.01 0.01; visual mesh filename=package://fetch_description/meshes/bucket.STL scale=0.01 0.01 0.01
Joints:
- added joint fetch_tool_fixed_joint: type fixed, parent gripper_link, child fetch_tool_link, origin xyz=-0.1 0 -0.195 rpy=0 1.5708 0

File: fetch_moveit_config/config/fetch.ros2_control.xacro (robot description, xacro)
@@ -4,9 +4,12 @@
         <xacro:property name="initial_positions" value="${load_yaml(initial_positions_file)['initial_positions']}"/>
         <ros2_control name="${name}" type="system">
-	     <hardware>
-                    <plugin>topic_based_ros2_control/TopicBasedSystem</plugin>
-                    <param name="joint_commands_topic">/isaac_joint_commands</param>
-                    <param name="joint_states_topic">/isaac_joint_states</param>
+            <hardware>
+                <plugin>topic_based_ros2_control/TopicBasedSystem</plugin>
+                <param name="joint_commands_topic">/isaac_joint_commands</param>
+                <param name="joint_states_topic">/joint_states</param>
             </hardware>
+            <!--hardware>
+            <plugin>mock_components/GenericSystem</plugin>
+            </hardware-->
             <joint name="shoulder_pan_joint">
                 <command_interface name="position"/>
